File: hardware/DPCM-map.kicad_pcb (KiCad board)
At the start: 2 copper layers, 178 x 178 mm, 98 parts, among them J1 JMP, J2 Conn_01x06_Male, J3 Touch_Pad_-, J4 Touch_Pad_0, J5 Touch_Pad_+, J6 JMP, J7 SSD1306, P1 USB_C_Plug, Q1 2N7002, Q2 2N7002, SW1 SW_Push, SW2 SW_+_Fb, SW3 SW_0_Fb, SW4 SW_-_Fb, U1 AZ1117-3.3, U2 BME280, U4 ESP32-WROOM-32, U5 CH340G, Y1 12MHz

Commit message: Aggiunti bottoni touch, rotti board edges
Parts:
- J3: value Touch_Pad_- -> Touch_Pad_+
- J5: value Touch_Pad_+ -> Touch_Pad_-
- J7: moved to B.Cu
- moved C1 240.8 mm to (33.9, 117.4), turned to 0 degrees
- moved C29 240.7 mm to (34.0, 119.0), turned to 0 degrees
- moved C34 240.7 mm to (34.0, 120.7), turned to 0 degrees
- moved J1 236.8 mm to (36.6, 134.0), turned to 180 degrees
- moved J6 235.8 mm to (36.6, 127.7), turned to 180 degrees
- moved U1 235.4 mm to (36.8, 113.0), turned to 0 degrees
- moved R3 231.6 mm to (39.3, 134.3), turned to 90 degrees
- moved C7 230.9 mm to (39.3, 131.2), turned to 90 degrees
- moved R6 230.4 mm to (39.3, 128.1), turned to 90 degrees
- moved C12 230.3 mm to (39.7, 108.5), turned to 0 degrees
- moved C17 230.1 mm to (39.3, 124.9), turned to 90 degrees
- moved C5 229.2 mm to (39.7, 117.4), turned to 180 degrees
- moved P1 184.6 mm to (113.5, 196.8), turned to 270 degrees
- moved SW1 183.9 mm to (115.5, 178.6), turned to 90 degrees
- moved J2 175.4 mm to (88.5, 142.5)
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Connections:
- D2 pad 2: (no net) -> Net-(D2-Pad2)
- J2 pad 1: (no net) -> Net-(J2-Pad1)
- J2 pad 2: (no net) -> Net-(J2-Pad2)
- P1 pad A5: (no net) -> Net-(P1-PadA5)
- P1 pad A8: (no net) -> Net-(P1-PadA8)
- P1 pad B5: (no net) -> Net-(P1-PadB5)
- P1 pad B8: (no net) -> Net-(P1-PadB8)
- U4 pad 10: (no net) -> Net-(U4-Pad10)
- U4 pad 11: (no net) -> Net-(U4-Pad11)
- U4 pad 12: (no net) -> Net-(U4-Pad12)
- U4 pad 17: (no net) -> Net-(U4-Pad17)
- U4 pad 18: (no net) -> Net-(U4-Pad18)
- U4 pad 19: (no net) -> Net-(U4-Pad19)
- U4 pad 20: (no net) -> Net-(U4-Pad20)
- U4 pad 21: (no net) -> Net-(U4-Pad21)
- U4 pad 22: (no net) -> Net-(U4-Pad22)
- U4 pad 24: (no net) -> Net-(U4-Pad24)
- U4 pad 27: (no net) -> Net-(U4-Pad27)
- U4 pad 28: (no net) -> Net-(U4-Pad28)
- U4 pad 29: (no net) -> Net-(U4-Pad29)
- U4 pad 30: (no net) -> Net-(U4-Pad30)
- U4 pad 31: (no net) -> Net-(U4-Pad31)
- U4 pad 32: (no net) -> Net-(U4-Pad32)
- U4 pad 37: (no net) -> Net-(U4-Pad37)
- U4 pad 4: (no net) -> Net-(U4-Pad4)
- U4 pad 5: (no net) -> Net-(U4-Pad5)
- U4 pad 6: (no net) -> Net-(U4-Pad6)
- U4 pad 7: (no net) -> Net-(U4-Pad7)
- U4 pad 8: (no net) -> Net-(U4-Pad8)
- U5 pad 10: (no net) -> Net-(U5-Pad10)
- U5 pad 11: (no net) -> Net-(U5-Pad11)
- U5 pad 12: (no net) -> Net-(U5-Pad12)
- U5 pad 15: (no net) -> Net-(U5-Pad15)
- U5 pad 9: (no net) -> Net-(U5-Pad9)
Routing:
- net TOUCH_0: vias 0 -> 56
- net TOUCH_-: vias 0 -> 49
- net TOUCH_+: vias 0 -> 49
- added copper zone on B.Cu, net TOUCH_+
- added copper zone on F.Cu, net TOUCH_+
- added copper zone on B.Cu, net TOUCH_-
- added copper zone on F.Cu, net TOUCH_-
- added copper zone on B.Cu, net TOUCH_0
- added copper zone on F.Cu, net TOUCH_0
Other:
- board text added: "Minimizzare le capacità parassite per i pulsanti touch (no ground fill)"
- board text added: "controllare distanza considerata vera lunghezza (clearance 1mm tra scheda e case, non va superata)"

Commit message: did some initial routing
Parts:
- added C41: 100n, Capacitor_SMD:C_0603_1608Metric, F.Cu at (144.0, 91.2)
- moved C29 224.1 mm to (254.3, 159.9)
- moved C34 160.7 mm to (194.6, 122.6), turned to 180 degrees
- moved C1 118.9 mm to (137.9, 175.0), turned to 90 degrees
- moved C3 117.8 mm to (261.4, 100.1)
- moved C17 116.6 mm to (137.5, 187.7), turned to 0 degrees
- moved JP3 115.6 mm to (215.9, 104.8)
- moved J6 113.5 mm to (134.6, 185.0), turned to 90 degrees
- moved J7 113.4 mm to (220.9, 107.4), turned to 0 degrees
- moved U1 113.3 mm to (133.5, 172.1), turned to 90 degrees
- moved JP1 112.5 mm to (216.1, 100.5)
- moved R6 112.2 mm to (134.3, 187.7), turned to 0 degrees
- moved C5 111.0 mm to (137.9, 169.2), turned to 270 degrees
- moved C12 107.9 mm to (129.0, 169.2), turned to 90 degrees
- moved C7 107.9 mm to (131.2, 187.7), turned to 0 degrees
- moved J1 105.0 mm to (128.4, 185.1), turned to 90 degrees
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Connections:
- D2 pad 2: Net-(D2-Pad2) -> (no net)
- J2 pad 1: Net-(J2-Pad1) -> (no net)
- J2 pad 2: Net-(J2-Pad2) -> (no net)
- P1 pad A5: Net-(P1-PadA5) -> (no net)
- P1 pad A8: Net-(P1-PadA8) -> (no net)
- P1 pad B5: Net-(P1-PadB5) -> (no net)
- P1 pad B8: Net-(P1-PadB8) -> (no net)
- U4 pad 10: Net-(U4-Pad10) -> (no net)
- U4 pad 11: Net-(U4-Pad11) -> (no net)
- U4 pad 12: Net-(U4-Pad12) -> (no net)
- U4 pad 17: Net-(U4-Pad17) -> (no net)
- U4 pad 18: Net-(U4-Pad18) -> (no net)
- U4 pad 19: Net-(U4-Pad19) -> (no net)
- U4 pad 20: Net-(U4-Pad20) -> (no net)
- U4 pad 21: Net-(U4-Pad21) -> (no net)
- U4 pad 22: Net-(U4-Pad22) -> (no net)
- U4 pad 24: Net-(U4-Pad24) -> (no net)
- U4 pad 27: Net-(U4-Pad27) -> (no net)
- U4 pad 28: Net-(U4-Pad28) -> (no net)
- U4 pad 29: Net-(U4-Pad29) -> (no net)
- U4 pad 30: Net-(U4-Pad30) -> (no net)
- U4 pad 31: Net-(U4-Pad31) -> (no net)
- U4 pad 32: Net-(U4-Pad32) -> (no net)
- U4 pad 37: Net-(U4-Pad37) -> (no net)
- U4 pad 4: Net-(U4-Pad4) -> (no net)
- U4 pad 5: Net-(U4-Pad5) -> (no net)
- U4 pad 6: Net-(U4-Pad6) -> (no net)
- U4 pad 7: Net-(U4-Pad7) -> (no net)
- U4 pad 8: Net-(U4-Pad8) -> (no net)
- U5 pad 10: Net-(U5-Pad10) -> (no net)
- U5 pad 11: Net-(U5-Pad11) -> (no net)
- U5 pad 12: Net-(U5-Pad12) -> (no net)
- U5 pad 15: Net-(U5-Pad15) -> (no net)
- U5 pad 9: Net-(U5-Pad9) -> (no net)
Routing:
- net +5V: track 0.00 -> 496.3 mm
- net GND: track 0.00 -> 47.2 mm, vias 0 -> 1
- net Net-(D13-Pad2): track 0.00 -> 32.4 mm
- net Net-(D15-Pad2): track 0.00 -> 24.5 mm
- net Net-(D3-Pad2): track 0.00 -> 22.2 mm
- net Net-(D11-Pad4): track 0.00 -> 21.7 mm
- net Net-(D16-Pad2): track 0.00 -> 21.6 mm
- net +3V3: track 0.00 -> 20.1 mm
- net Net-(D14-Pad2): track 0.00 -> 20.0 mm
- net Net-(D5-Pad2): track 0.00 -> 19.5 mm
- net Net-(D7-Pad2): track 0.00 -> 18.8 mm
- net Net-(D11-Pad2): track 0.00 -> 16.0 mm
- net D-: track 0.00 -> 14.8 mm
- net D+: track 0.00 -> 14.5 mm
- net Net-(C16-Pad2): track 0.00 -> 13.9 mm, vias 0 -> 2
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Other:
- net class Default: trace_width 0.25 -> 0.35
- net class PWR added: clearance 0.2, trace_width 0.65, via_dia 0.8, via_drill 0.4

Commit message: first routing try
Parts:
- C2: value 1u -> 10u
- moved C6 52.4 mm to (215.1, 110.0)
- moved C3 49.3 mm to (212.0, 101.5), turned to 180 degrees
- moved C13 45.0 mm to (215.1, 101.5)
- moved J2 18.8 mm to (153.6, 129.8), turned to 180 degrees
- moved JP1 7.38 mm to (215.9, 107.9)
- moved C38 7.12 mm to (225.8, 145.0), turned to 90 degrees
- moved C40 6.33 mm to (226.4, 159.2), turned to 180 degrees
- moved C28 5.29 mm to (207.6, 121.1), turned to 180 degrees
- moved C27 4.46 mm to (212.4, 208.0), turned to 90 degrees
- moved D18 1.28 mm to (206.2, 118.1), turned to 180 degrees
- moved JP3 1.12 mm to (215.9, 103.6)
- moved D6 0.54 mm to (222.1, 145.2), turned to 180 degrees
- moved D1 0.11 mm to (215.3, 206.8), turned to 90 degrees
- turned D4 to 180 degrees
Routing:
- net +3V3: track 20.1 -> 288.5 mm, vias 0 -> 4
- net TOUCH_+: track 0.00 -> 189.5 mm, vias 49 -> 50
- net SCL: track 0.00 -> 183.9 mm, vias 0 -> 4
- net SDA: track 0.00 -> 181.4 mm, vias 0 -> 2
- net TOUCH_0: track 0.00 -> 139.3 mm, vias 56 -> 57
- net TX: track 10.3 -> 117.7 mm, vias 0 -> 2
- net LDR: track 0.00 -> 105.3 mm, vias 0 -> 1
- net RX: track 10.9 -> 116.1 mm, vias 0 -> 2
- net TOUCH_-: track 0.00 -> 104.6 mm, vias 49 -> 50
- net +5V: track 496.3 -> 588.2 mm
- net LED_CHAIN: track 0.00 -> 87.9 mm, vias 0 -> 2
- net BOOT0: track 0.00 -> 85.2 mm, vias 0 -> 1
- net Net-(D22-Pad2): track 0.00 -> 72.0 mm
- net WIFI_RESET: track 0.00 -> 60.3 mm, vias 0 -> 2
- net EN: track 0.00 -> 57.8 mm, vias 0 -> 1
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